File: PCB/PCB.kicad_pcb (KiCad board)
At the start: 2 copper layers, 107 x 80 mm, 65 parts, among them J1 Conn_01x10, J2 Conn_01x10, J3 BATT, J4 Speaker, J5 XKB_PJ-342B, M1 ModuleNC, SW1 SW_SPDT_G, U1 LM358DR2G, U2 XIAO RA4M1, U3 AMS1117-5.0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

Commit message: add files
Parts:
- R18: value 220R -> 10K
- moved C15 19.5 mm to (239.6, 174.4)
Connections:
- U3 pad 2: Net-(D1-K) -> +5V
- U3 pad 3: +5V -> Net-(D1-K)
Routing:
- net GNDD: track 530.2 -> 535.5 mm
- net Net-(D1-K): track 14.6 -> 12.1 mm
- net +5V: track 157.9 -> 160.0 mm
Changed lines of the file:
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@@
 	(footprint "Capacitor_SMD:C_0603_1608Metric"
 		(layer "F.Cu")
-		(at 240.775 154.9 180)
+		(at 239.55 174.4 180)
 		(descr "Capacitor SMD 0603 (1608 Metric), square (rectangular) end terminal, IPC_7351 nominal, (Body size source: IPC-SM-782 page 76, https://www.pcb-3d.com/wordpress/wp-content/uploads/ipc-sm-782a_amendment_1_and_2.pdf), generated with kicad-footprint-generator")
 		(tags "capacitor")
@@
 			(layers "F.Cu" "F.Paste" "F.Mask")
 			(roundrect_rratio 0.25)
-			(net 4 "Net-(D1-K)")
+			(net 45 "+5V")
 			(pinfunction "VO")
 			(pintype "power_out")
@@
 			(layers "F.Cu" "F.Paste" "F.Mask")
 			(roundrect_rratio 0.25)
-			(net 4 "Net-(D1-K)")
+			(net 45 "+5V")
 			(pinfunction "VO")
 			(pintype "power_out")
@@
 			(layers "F.Cu" "F.Paste" "F.Mask")
 			(roundrect_rratio 0.25)
-			(net 45 "+5V")
+			(net 4 "Net-(D1-K)")
 			(pinfunction "VI")
 			(pintype "power_in")
@@
 		)
 		(property "Value" "XKB_PJ-342B"
-			(at 3.5 6 360)
+			(at 3.5 6 0)
 			(layer "F.Fab")
 			(effects
@@
 			)
 		)
-		(property "Value" "220R"
+		(property "Value" "10K"
 			(at 0 1.5 0)
 			(layer "F.Fab")
@@
 	)
 	(segment
+		(start 238.775 174.4)
+		(end 237.05 174.4)
+		(width 0.4)
+		(layer "F.Cu")
+		(net 1)
+	)
+	(segment
 		(start 178.05 133.4)
 		(end 177.4 133.4)
@@
 	)
 	(segment
+		(start 237.05 174.4)
+		(end 237.05 173.4)
+		(width 0.4)
+		(layer "F.Cu")
+		(net 1)
+	)
+	(segment
 		(start 167.65 179.3)
 		(end 167.55 179.4)
@@
 	)
 	(segment
+		(start 234.59 173.48)
+		(end 236.97 173.48)
+		(width 0.4)
+		(layer "F.Cu")
+		(net 1)
+	)
+	(segment
 		(start 154.875 174.35)
 		(end 154.825 174.4)
@@
 	)
 	(segment
+		(start 237.05 173.4)
+		(end 236.97 173.48)
+		(width 0.4)
+		(layer "F.Cu")
+		(net 1)
+	)
+	(segment
 		(start 154.875 159.9)
 		(end 154.875 164.005)
@@
 	)
 	(segment
-		(start 241.55 169.05)
-		(end 241.55 164.55)
+		(start 243.85 164.55)
+		(end 243.85 168.1)
+		(width 0.8)
+		(layer "F.Cu")
+		(net 4)
+	)
+	(segment
+		(start 243.85 168.1)
+		(end 242.55 169.4)
 		(width 0.8)
 		(layer "F.Cu")
@@
 	(segment
 		(start 241.2 169.4)
-		(end 241.55 169.05)
+		(end 241.2 173.525)
 		(width 0.8)
 		(layer "F.Cu")
@@
 	)
 	(segment
-		(start 241.55 158.25)
-		(end 241.55 154.9)
+		(start 242.55 169.4)
+		(end 241.2 169.4)
 		(width 0.8)
 		(layer "F.Cu")
@@
 	)
 	(segment
-		(start 241.55 164.55)
-		(end 241.55 158.25)
+		(start 241.2 173.525)
+		(end 240.325 174.4)
 		(width 0.8)
 		(layer "F.Cu")
@@
 	)
 	(segment
-		(start 204.1 124.9)
-		(end 205.55 124.9)
+		(start 241.325 151.4)
+		(end 244.55 151.4)
 		(width 0.8)
 		(layer "F.Cu")
@@
 	)
 	(segment
-		(start 241.325 152.125)
-		(end 240.55 152.9)
+		(start 204.1 124.9)
+		(end 205.55 124.9)
 		(width 0.8)
 		(layer "F.Cu")
@@
 	)
 	(segment
-		(start 241.325 147.975)
-		(end 241.4 147.9)
+		(start 229.55 148.4)
+		(end 220.55 148.4)
 		(width 0.8)
 		(layer "F.Cu")
@@
 	)
 	(segment
-		(start 229.55 148.4)
-		(end 220.55 148.4)
-		(width 0.8)
-		(layer "F.Cu")
-		(net 45)
-	)
-	(segment
 		(start 241.4 147.9)
 		(end 244.55 147.9)
@@
 	)
 	(segment
-		(start 234.05 152.9)
-		(end 229.55 148.4)
-		(width 0.8)
-		(layer "F.Cu")
-		(net 45)
-	)
-	(segment
-		(start 241.325 151.4)
-		(end 241.325 152.125)
-		(width 0.8)
-		(layer "F.Cu")
-		(net 45)
-	)
-	(segment
 		(start 229.275 108.9)
 		(end 214.05 108.9)
@@
 	)
 	(segment
-		(start 244.67 147.9)
-		(end 244.67 151.4)
+		(start 244.55 151.4)
+		(end 244.55 153.9)
 		(width 0.8)
 		(layer "F.Cu")
@@
 	)
 	(segment
-		(start 241.325 151.4)
-		(end 244.67 151.4)
-		(width 0.8)
-		(layer "F.Cu")
-		(net 45)
-	)
-	(segment
 		(start 229.275 108.9)
 		(end 229.275 112.35)
@@
 	)
 	(segment
+		(start 220.55 148.4)
+		(end 207.55 135.4)
+		(width 0.8)
+		(layer "F.Cu")
+		(net 45)
+	)
+	(segment
 		(start 188.225 122.4)
 		(end 185.55 122.4)
@@
 	)
 	(segment
-		(start 244.67 151.4)
-		(end 244.67 163.73)
+		(start 244.67 143.28)
+		(end 244.55 143.4)
 		(width 0.8)
 		(layer "F.Cu")
@@
 	)
 	(segment
-		(start 244.67 163.73)
-		(end 243.85 164.55)
+		(start 241.55 158.25)
+		(end 239.4 158.25)
 		(width 0.8)
 		(layer "F.Cu")
@@
 	)
 	(segment
-		(start 244.67 141.565)
-		(end 244.67 147.9)
+		(start 241.55 156.9)
+		(end 244.55 153.9)
 		(width 0.8)
 		(layer "F.Cu")
@@
 	)
 	(segment
-		(start 184.55 118.4)
-		(end 183.915 117.765)
+		(start 244.55 143.4)
+		(end 244.55 147.9)
 		(width 0.8)
 		(layer "F.Cu")
@@
 	)
 	(segment
-		(start 220.55 148.4)
-		(end 207.55 135.4)
+		(start 184.55 118.4)
+		(end 183.915 117.765)
 		(width 0.8)
 		(layer "F.Cu")
@@
 	)
 	(segment
-		(start 240.55 152.9)
-		(end 234.05 152.9)
+		(start 244.67 141.565)
+		(end 244.67 143.28)
 		(width 0.8)
 		(layer "F.Cu")
@@
 	)
 	(segment
-		(start 244.55 147.9)
-		(end 244.67 147.9)
+		(start 241.55 158.25)
+		(end 241.55 156.9)
 		(width 0.8)
 		(layer "F.Cu")
@@
 		(width 0.8)
 		(layer "F.Cu")
+		(net 45)
+	)
+	(segment
+		(start 241.55 164.55)
+		(end 241.55 158.25)
+		(width 0.8)
+		(layer "F.Cu")
+		(net 45)
+	)
+	(segment
+		(start 244.55 147.9)
+		(end 244.55 151.4)
+		(width 0.8)
+		(layer "F.Cu")
+		(net 45)
+	)
+	(segment
+		(start 241.325 147.975)
+		(end 241.4 147.9)
+		(width 0.8)
+		(layer "F.Cu")
+		(net 45)
+	)
+	(segment
+		(start 239.4 158.25)
+		(end 229.55 148.4)
+		(width 0.8)
+		(layer "F.Cu")
