File: PCB/PCB.kicad_sch (KiCad schematic)
At the start: 65 parts, among them J1 Conn_01x10, J2 Conn_01x10, J3 BATT, J4 Speaker, J5 XKB_PJ-342B, M1 ModuleNC, SW1 SW_SPDT_G, U1 LM358DR2G, U2 XIAO RA4M1, U3 AMS1117-5.0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

Commit message: add files
Parts:
- R18: value 220R -> 10K
Connections:
- net +5V: now also U3.2 (VO); no longer U3.3 (VI)
- net at C15.1, D1.1 (K): now also U3.3 (VI); no longer U3.2 (VO)
Changed lines of the file:
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@@
 	)
 	(junction
-		(at 219.71 123.19)
+		(at 243.84 123.19)
 		(diameter 0)
 		(color 0 0 0 0)
@@
 	)
 	(junction
+		(at 219.71 123.19)
+		(diameter 0)
+		(color 0 0 0 0)
+	)
+	(junction
 		(at 279.4 59.69)
 		(diameter 0)
@@
 	)
 	(junction
-		(at 243.84 123.19)
-		(diameter 0)
-		(color 0 0 0 0)
-	)
-	(junction
 		(at 218.44 57.15)
 		(diameter 0)
@@
 	(wire
 		(pts
+			(xy 219.71 123.19) (xy 219.71 142.24)
+		)
+		(stroke
+			(width 0)
+			(type default)
+		)
+	)
+	(wire
+		(pts
 			(xy 237.49 87.63) (xy 237.49 91.44)
 		)
@@
 	(wire
 		(pts
+			(xy 236.22 123.19) (xy 243.84 123.19)
+		)
+		(stroke
+			(width 0)
+			(type default)
+		)
+	)
+	(wire
+		(pts
 			(xy 279.4 240.03) (xy 281.94 240.03)
 		)
@@
 	(wire
 		(pts
-			(xy 219.71 123.19) (xy 220.98 123.19)
-		)
-		(stroke
-			(width 0)
-			(type default)
-		)
-	)
-	(wire
-		(pts
 			(xy 279.4 168.91) (xy 281.94 168.91)
 		)
@@
 	(wire
 		(pts
-			(xy 219.71 142.24) (xy 219.71 123.19)
+			(xy 219.71 113.03) (xy 219.71 123.19)
 		)
 		(stroke
@@
 	(wire
 		(pts
+			(xy 219.71 123.19) (xy 220.98 123.19)
+		)
+		(stroke
+			(width 0)
+			(type default)
+		)
+	)
+	(wire
+		(pts
 			(xy 95.25 116.84) (xy 123.19 116.84)
 		)
@@
 	(wire
 		(pts
-			(xy 236.22 123.19) (xy 243.84 123.19)
-		)
-		(stroke
-			(width 0)
-			(type default)
-		)
-	)
-	(wire
-		(pts
 			(xy 207.01 57.15) (xy 209.55 57.15)
 		)
@@
 	(wire
 		(pts
-			(xy 219.71 113.03) (xy 219.71 123.19)
-		)
-		(stroke
-			(width 0)
-			(type default)
-		)
-	)
-	(wire
-		(pts
 			(xy 143.51 219.71) (xy 143.51 162.56)
 		)
@@
 		(lib_id "Regulator_Linear:AMS1117-5.0")
 		(at 228.6 123.19 0)
+		(mirror y)
 		(unit 1)
 		(exclude_from_sim no)
@@
 		(on_board yes)
 		(dnp no)
-		(fields_autoplaced yes)
 		(property "Reference" "U3"
 			(at 228.6 116.84 0)
@@
 		)
 		(property "Datasheet" "http://www.advanced-monolithic.com/pdf/ds1117.pdf"
-			(at 231.14 129.54 0)
+			(at 226.06 129.54 0)
 			(effects
 				(font
@@
 			)
 		)
-		(property "Value" "220R"
+		(property "Value" "10K"
 			(at 251.46 87.63 90)
 			(effects
